Commit message: Ready to submit. Photos are needed to be attached

File: my_robot/urdf/my_robot.xacro (robot description, xacro)
@@ -1,132 +1,100 @@
-<?xml version="1.0"?>
+<?xml version='1.0'?>
 <robot name="my_robot" xmlns:xacro="http://www.ros.org/wiki/xacro">
-<xacro:include filename="$(find my_robot)/urdf/my_robot.gazebo" />
-  <!--Links-->
+  <xacro:include filename="$(find my_robot)/urdf/my_robot.gazebo" />
   <link name="robot_footprint"></link>
   <joint name="robot_footprint_joint" type="fixed">
     <origin xyz="0 0 0" rpy="0 0 0" />
-    <parent link="robot_footprint" />
+    <parent link="robot_footprint"/>
     <child link="chassis" />
   </joint>
-  <link name="chassis">
+  <link name='chassis'>
     <pose>0 0 0.1 0 0 0</pose>
     <inertial>
-      <mass value="5.0" />
-      <origin xyz="0 0 0" rpy="0 0 0" />
+      <mass value="15.0"/>
+      <origin xyz="0.0 0 0" rpy=" 0 0 0"/>
       <inertia
-        ixx="0.1" ixy="0" ixz="0"
-        iyy="0.1" iyz="0"
-        izz="0.1" />
+          ixx="0.1" ixy="0" ixz="0"
+          iyy="0.1" iyz="0"
+          izz="0.1"
+      />
     </inertial>
-    <collision name="box_collision">
-      <origin xyz="0 0 0.05" rpy="0 0 0" />
+    <collision name='collision'>
+      <origin xyz="0 0 0" rpy=" 0 0 0"/>
       <geometry>
-        <box size=".4 .2 .1" />
+        <box size=".4 .2 .1"/>
       </geometry>
     </collision>
-    <visual name="box_visual">
-      <origin xyz="0 0 0.05" rpy="0 0 0" />
+    <visual name='chassis_visual'>
+      <origin xyz="0 0 0" rpy=" 0 0 0"/>
       <geometry>
-        <box size=".4 .2 .1" />
+        <box size=".4 .2 .1"/>
       </geometry>
     </visual>
-    <collision name="cylinder_colllision">
-      <origin xyz="0.075 0 0.125" rpy="0 0 0" />
+    <collision name='back_caster_collision'>
+      <origin xyz="-0.15 0 -0.05" rpy=" 0 0 0"/>
       <geometry>
-        <cylinder radius=".15" length=".05" />
+        <sphere radius="0.0499"/>
       </geometry>
     </collision>
-    <visual name="cylinder_visual">
-      <origin xyz="0.075 0 0.125" rpy="0 0 0" />
+    <visual name='back_caster_visual'>
+      <origin xyz="-0.15 0 -0.05" rpy=" 0 0 0"/>
       <geometry>
-        <cylinder radius=".15" length=".05" />
+        <sphere radius="0.05"/>
+      </geometry>
+    </visual>
+    <collision name='front_caster_collision'>
+      <origin xyz="0.15 0 -0.05" rpy=" 0 0 0"/>
+      <geometry>
+        <sphere radius="0.0499"/>
+      </geometry>
+    </collision>
+    <visual name='front_caster_visual'>
+      <origin xyz="0.15 0 -0.05" rpy=" 0 0 0"/>
+      <geometry>
+        <sphere radius="0.05"/>
       </geometry>
     </visual>
   </link>
-  <link name="front_wheel_left">
+  <link name="left_wheel">
     <inertial>
-      <mass value="1.0" />
-      <origin xyz="0 0.01 0" rpy="0 1.5707 1.5707" />
+      <mass value="5.0"/>
+      <origin xyz="0.0 0 0" rpy=" 0 0 0"/>
       <inertia
-        ixx="0.1" ixy="0" ixz="0"
-        iyy="0.1" iyz="0"
-        izz="0.1" />
+          ixx="0.1" ixy="0" ixz="0"
+          iyy="0.1" iyz="0"
+          izz="0.1"/>
     </inertial>
-    <collision name="front_wheel_left_collision">
-      <origin xyz="0 0.01 0" rpy="0 1.5707 1.5707" />
+    <collision name='left_wheel_collision'>
+      <origin xyz="0 0 0" rpy=" 0 1.5707 1.5707"/>
       <geometry>
-        <cylinder radius="0.05" length="0.02" />
+        <cylinder radius="0.1" length="0.05" />
       </geometry>
     </collision>
-    <visual name="front_wheel_left_visual">
-      <origin xyz="0 0.01 0" rpy="0 1.5707 1.5707" />
+    <visual name='left_wheel_visual'>
+      <origin xyz="0 0 0" rpy=" 0 1.5707 1.5707"/>
       <geometry>
-        <cylinder radius="0.05" length="0.02" />
+        <cylinder radius="0.1" length="0.05" />
       </geometry>
     </visual>
   </link>
-  <link name="front_wheel_right">
-    <inertial>
-      <mass value="1.0" />
-      <origin xyz="0 -0.01 0" rpy="0 1.5707 1.5707" />
+  <link name="right_wheel">
+  <inertial>
+      <mass value="5.0"/>
+      <origin xyz="0.0 0 0" rpy=" 0 0 0"/>
       <inertia
-        ixx="0.1" ixy="0" ixz="0"
-        iyy="0.1" iyz="0"
-        izz="0.1" />
+          ixx="0.1" ixy="0" ixz="0"
+          iyy="0.1" iyz="0"
+          izz="0.1"/>
     </inertial>
-    <collision name="front_wheel_right_collision">
-      <origin xyz="0 -0.01 0" rpy="0 1.5707 1.5707" />
+    <collision name='right_wheel_collision'>
+      <origin xyz="0 0 0" rpy=" 0 1.5707 1.5707"/>
       <geometry>
-        <cylinder radius="0.05" length="0.02" />
+        <cylinder radius="0.1" length="0.05" />
       </geometry>
     </collision>
-    <visual name="front_wheel_right_visual">
-      <origin xyz="0 -0.01 0" rpy="0 1.5707 1.5707" />
+    <visual name='right_wheel_visual'>
+      <origin xyz="0 0 0" rpy=" 0 1.5707 1.5707"/>
       <geometry>
-        <cylinder radius="0.05" length="0.02" />
-      </geometry>
-    </visual>
-  </link>
-  <link name="rear_wheel_left">
-    <inertial>
-      <mass value="1.0" />
-      <origin xyz="0 0.01 0" rpy="0 1.5707 1.5707" />
-      <inertia
-        ixx="0.1" ixy="0" ixz="0"
-        iyy="0.1" iyz="0"
-        izz="0.1" />
-    </inertial>
-    <collision name="rear_wheel_left_collision">
-      <origin xyz="0 0.01 0" rpy="0 1.5707 1.5707" />
-      <geometry>
-        <cylinder radius="0.05" length="0.02" />
-      </geometry>
-    </collision>
-    <visual name="rear_wheel_left_visual">
-      <origin xyz="0 0.01 0" rpy="0 1.5707 1.5707" />
-      <geometry>
-        <cylinder radius="0.05" length="0.02" />
-      </geometry>
-    </visual>
-  </link>
-  <link name="rear_wheel_right">
-    <inertial>
-      <mass value="1.0" />
-      <origin xyz="0 -0.01 0" rpy="0 1.5707 1.5707" />
-      <inertia
-        ixx="0.1" ixy="0" ixz="0"
-        iyy="0.1" iyz="0"
-        izz="0.1" />
-    </inertial>
-    <collision name="rear_wheel_right_collision">
-      <origin xyz="0 -0.01 0" rpy="0 1.5707 1.5707" />
-      <geometry>
-        <cylinder radius="0.05" length="0.02" />
-      </geometry>
-    </collision>
-    <visual name="rear_wheel_right_visual">
-      <origin xyz="0 -0.01 0" rpy="0 1.5707 1.5707" />
-      <geometry>
-        <cylinder radius="0.05" length="0.02" />
+        <cylinder radius="0.1" length="0.05" />
       </geometry>
     </visual>
@@ -176,4 +144,32 @@
     </visual>
   </link>
+  <joint type="continuous" name="left_wheel_hinge">
+    <origin xyz="0 0.15 0" rpy="0 0 0"/>
+    <child link="left_wheel"/>
+    <parent link="chassis"/>
+    <axis xyz="0 1 0" rpy="0 0 0"/>
+    <limit effort="10000" velocity="1000"/>
+    <dynamics damping="1.0" friction="1.0"/>
+  </joint>
+  <joint type="continuous" name="right_wheel_hinge">
+    <origin xyz="0 -0.15 0" rpy="0 0 0"/>
+    <child link="right_wheel"/>
+    <parent link="chassis"/>
+    <axis xyz="0 1 0" rpy="0 0 0"/>
+    <limit effort="10000" velocity="1000"/>
+    <dynamics damping="1.0" friction="1.0"/>
+  </joint>
+  <joint type="fixed" name="camera_joint">
+    <origin xyz="0.2 0 0.0" rpy="0 0 0" />
+    <axis xyz="0 1 0" rpy="0 0 0" />
+    <parent link="chassis" />
+    <child link="camera" />
+  </joint>
+  <joint name="hokuyo_fixed" type="fixed">
+    <origin xyz="0.15 0 0.1" rpy="0 0 0"/>
+    <axis xyz="0 1 0" rpy="0 0 0"/>
+    <parent link="chassis" />
+    <child link="hokuyo" />
+  </joint>
   <!--Colors-->
   <gazebo reference="chassis">
@@ -183,60 +179,9 @@
     <material>Gazebo/Red</material>
   </gazebo>
-  <gazebo reference="front_wheel_right">
+  <gazebo reference="right_wheel">
     <material>Gazebo/Black</material>
   </gazebo>
-  <gazebo reference="rear_wheel_left">
+  <gazebo reference="left_wheel">
     <material>Gazebo/Black</material>
   </gazebo>
-  <gazebo reference="rear_wheel_right">
-    <material>Gazebo/Black</material>
-  </gazebo>
-  <gazebo reference="front_wheel_left">
-    <material>Gazebo/Black</material>
-  </gazebo>
-  <!--Joints-->
-  <joint type="continuous" name="joint_front_wheel_left">
-    <origin xyz=".15 0.1 0" rpy="0 0 0" />
-    <child link="front_wheel_left" />
-    <parent link="chassis" />
-    <axis xyz="0 1 0" rpy="0 0 0" />
-    <limit effort="10000" velocity="1000" />
-    <dynamics damping="1.0" friction="1.0" />
-  </joint>
-  <joint type="continuous" name="joint_front_wheel_right">
-    <origin xyz=".15 -0.1 0" rpy="0 0 0" />
-    <child link="front_wheel_right" />
-    <parent link="chassis" />
-    <axis xyz="0 1 0" rpy="0 0 0" />
-    <limit effort="10000" velocity="1000" />
-    <dynamics damping="1.0" friction="1.0" />
-  </joint>
-  <joint type="continuous" name="joint_rear_wheel_left">
-    <origin xyz="-0.15 0.1 0" rpy="0 0 0" />
-    <child link="rear_wheel_left" />
-    <parent link="chassis" />
-    <axis xyz="0 1 0" rpy="0 0 0" />
-    <limit effort="10000" velocity="1000" />
-    <dynamics damping="1.0" friction="1.0" />
-  </joint>
-  <joint type="continuous" name="joint_rear_wheel_right">
-    <origin xyz="-0.15 -0.1 0" rpy="0 0 0" />
-    <child link="rear_wheel_right" />
-    <parent link="chassis" />
-    <axis xyz="0 1 0" rpy="0 0 0" />
-    <limit effort="10000" velocity="1000" />
-    <dynamics damping="1.0" friction="1.0" />
-  </joint>
-  <joint type="fixed" name="camera_joint">
-    <origin xyz="0.22 0 0.07" rpy="0 0 0" />
-    <axis xyz="0 1 0" rpy="0 0 0" />
-    <parent link="chassis" />
-    <child link="camera" />
-  </joint>
-  <joint name="hokuyo_fixed" type="fixed">
-    <origin xyz="0.15 0 0.175" rpy="0 0 0"/>
-    <axis xyz="0 1 0" rpy="0 0 0"/>
-    <parent link="chassis" />
-    <child link="hokuyo" />
-  </joint>
 </robot>

Commit message: the maping package works fine now

File: my_robot/urdf/my_robot.xacro (robot description, xacro)
@@ -144,4 +144,11 @@
     </visual>
   </link>
+  <joint name="camera_optical_joint" type="fixed">
+    <origin xyz="0 0 0" rpy="-1.5707 0 -1.5707"/>
+    <parent link="camera"/>
+    <child link="camera_link_optical"/>
+  </joint>
+  <link name="camera_link_optical">
+  </link>
   <joint type="continuous" name="left_wheel_hinge">
     <origin xyz="0 0.15 0" rpy="0 0 0"/>
